File: ECGampl/ECGampl.brd (EAGLE design)
At the start: 67 x 45.7 mm, 19 parts, among them U1 AD624ADZ

Commit message: successful routing
Routing:
- net N$18: track 0.00 -> 58.6 mm
- net VSS: track 0.00 -> 56.7 mm
- net N$13: track 0.00 -> 48.8 mm
- net N$12: track 0.00 -> 41.5 mm
- net VDD: track 0.00 -> 37.4 mm
- net IN2: track 0.00 -> 20.7 mm
- net N$9: track 0.00 -> 20.3 mm
- net N$6: track 0.00 -> 15.0 mm
- net N$7: track 0.00 -> 12.4 mm
- net N$5: track 0.00 -> 11.7 mm
- net N$1: track 0.00 -> 10.9 mm
- net N$2: track 0.00 -> 10.7 mm
- net N$4: track 0.00 -> 7.78 mm
- net IN1: track 0.00 -> 7.72 mm
- added copper zone on layer 16, net GND
